File: circuit/ESP_Racer_2025/ESP_Racer_2025.kicad_pcb (KiCad board)
At the start: 2 copper layers, 20 x 35 mm, 19 parts, among them IC1 XCL102D333CR-G, J1 Conn_LED_1, J2 Conn_LED_2, J3 Conn_Servo, U1 DRV8835DSST, U2 SFV12R-2STE1LF, U3 ESP32-C3-WROOM-02

Commit message: pcb fix
Parts:
- J1, J2: footprint JST_ZH_B2B-ZR_1x02_P1.50mm_Vertical:JST_ZH_B2B-ZR_1x02_P1.50mm_Vertical -> Molex:Molex_PicoBlade_53047-0210_1x02_P1.25mm_Vertical
- J3: footprint JST_ZH_B3B-ZR_1x03_P1.50mm_Vertical:JST_ZH_B3B-ZR_1x03_P1.50mm_Vertical -> Molex:Molex_PicoBlade_53047-0310_1x03_P1.25mm_Vertical
- R6: value 10k -> 20k
- moved C4 0.85 mm to (143.5, 80.9)
- moved J3 0.81 mm to (147.0, 91.0)
- moved J1 0.74 mm to (141.0, 92.0)
- moved J2 0.74 mm to (135.5, 92.0)
- moved D1 0.28 mm to (136.1, 81.4)
- moved C5 0.08 mm to (147.1, 82.5)
- moved R4 0.08 mm to (147.1, 84.0)
- moved R5 0.08 mm to (147.1, 81.0)
- moved R6 0.08 mm to (147.1, 85.5)
- turned C2 to 90 degrees
Connections:
- C2 pad 2: Net-(U1-VCC) -> GND
- C3 pad 2: Net-(U1-VM) -> GND
- U1 pad 1: Net-(U1-VM) -> +BATT
- U1 pad 12: Net-(U1-VCC) -> +3.3V
- U3 pad 16: AIN 1 -> unconnected-(U3-GPIO2/ADC1_CH2/FSPIQ-Pad16)
- U3 pad 17: Servo_PWM -> AIN 1
- U3 pad 5: unconnected-(U3-GPIO6/FSPICLK/MTCK-Pad5) -> Servo_PWM
Routing:
- net Servo_PWM: track 22.8 -> 33.8 mm
- net GND: track 94.6 -> 102.2 mm, vias 10 -> 9
- net +3.3V: track 38.5 -> 41.7 mm, vias 0 -> 2
- net Net-(U1-VCC): track 2.07 -> 0.00 mm
- net Net-(U1-VM): track 1.29 -> 0.00 mm
- net Net-(J1-Pin_1): track 2.69 -> 3.93 mm
- net Motor_B: track 6.81 -> 7.79 mm
- net +BATT: track 42.0 -> 43.0 mm
- net AIN 1: track 26.5 -> 27.4 mm
- net Net-(J2-Pin_1): track 3.41 -> 4.15 mm

Commit message: fix pcb
Parts:
- moved J2 0.20 mm to (135.7, 92.0)
Routing:
- net GND: track 102.2 -> 106.3 mm, vias 9 -> 11
- net +BATT: track 43.0 -> 44.9 mm
- net Net-(IC1-CE): track 2.48 -> 3.45 mm
