File: circuit/ESP_Racer_2025/ESP_Racer_2025.kicad_pcb (KiCad board)
At the start: 2 copper layers, 20 x 35 mm, 23 parts, among them IC1 XCL102D333CR-G, J1 Conn_LED_1, J2 Conn_LED_2, J3 Conn_Servo, J4 Conn_USB, Q3 IRLML6402, U1 DRV8835DSST, U2 SFV12R-2STE1LF, U3 ESP32-C3-WROOM-02

Commit message: fix pcb
Routing:
- net GND: track 107.6 -> 120.5 mm, vias 11 -> 14
- net LED_2: track 23.4 -> 27.6 mm
- net Servo_PWM: track 33.4 -> 35.7 mm

Commit message: fix pcb
Routing:
- net GND: track 120.5 -> 118.8 mm, vias 14 -> 50
- net Net-(U3-EN): track 18.5 -> 19.9 mm

Commit message: pcb update
Routing:
- net GND: track 118.8 -> 121.9 mm, vias 50 -> 51
